File: devboard/fpchp.kicad_sch (KiCad schematic)
At the start: 15 parts, among them J1 FPC Connector

Commit message: hp adapter rev.2
Parts:
- CP1, CP2: now not fitted
Changed lines of the file:
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@@
 		(in_bom yes)
 		(on_board yes)
-		(dnp no)
+		(dnp yes)
 		(property "Reference" "CP2"
 			(at 142.24 127 0)
@@
 		(in_bom yes)
 		(on_board yes)
-		(dnp no)
+		(dnp yes)
 		(property "Reference" "CP1"
 			(at 133.985 127 0)
