File: devboard/devboard.kicad_sch (KiCad schematic)
At the start: 17 parts, among them J1 IC1F-68RD-1.27SF(52), J2 92140-010LF, J3 D_{0-15}, J4 A_{0-15}, J5 A_{16-25} IOIS16 RESET WE IOR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, J6 IREQ STSHG SPKR WAIT REG CE_{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, J7 REG RESET IREQ IOWR IORD OE C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, SW1 CD1, SW2 CD2

Commit message: pld, docs
Parts:
- JP2: value CD1 -> CD2
- JP3: value CD2 -> CD1
Other:
- note added: "P1=J4 J=CLK2 P2=J5 K=CLK3 P3=J3 L=CLK1 P4=J6 M=CLK4"
Changed lines of the file:
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@@
 		)
 	)
+	(text "P1=J4 J=CLK2\nP2=J5 K=CLK3\nP3=J3 L=CLK1\nP4=J6 M=CLK4"
+		(exclude_from_sim no)
+		(at 117.348 68.326 0)
+		(effects
+			(font
+				(size 1.27 1.27)
+			)
+		)
+	)
 	(label "CLK3"
 		(at 168.91 87.63 0)
@@
 			)
 		)
-		(property "Value" "CD2"
+		(property "Value" "CD1"
 			(at 264.16 105.41 0)
 			(effects
@@
 			)
 		)
-		(property "Value" "CD1"
+		(property "Value" "CD2"
 			(at 264.16 102.87 0)
 			(effects

Commit message: devboard test
Connections:
- net CLK1: now also J7.13 (IO7); no longer J7.12 (IO8)
- net CLK3: now also J7.18 (IO2); no longer J7.13 (IO7)
- net CLK4: now also J7.12 (IO8); no longer J7.18 (IO2)
Other:
- note added: "P1=J4 J=CLK2 A_{0-15} P2=J5 K=CLK3 A_{16-25} IOIS16 RESET WE IORD OE IOWR P3=J3 L=CLK1 D_{0-15} P4=J6 M=CLK4 IREQ STSHG SPKR WAIT REG CE_{1,2} VS_{1,2} CD_{1,2} AUX_{1,4}"
- note removed: "P1=J4 J=CLK2 P2=J5 K=CLK3 P3=J3 L=CLK1 P4=J6 M=CLK4"
Changed lines of the file:
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@@
 		)
 	)
-	(text "P1=J4 J=CLK2\nP2=J5 K=CLK3\nP3=J3 L=CLK1\nP4=J6 M=CLK4"
+	(text "P1=J4 J=CLK2 A_{0-15}\nP2=J5 K=CLK3 A_{16-25} IOIS16 RESET WE IORD OE IOWR\nP3=J3 L=CLK1 D_{0-15}\nP4=J6 M=CLK4 IREQ STSHG SPKR WAIT REG CE_{1,2} VS_{1,2} CD_{1,2} AUX_{1,4}"
 		(exclude_from_sim no)
-		(at 117.348 68.326 0)
-		(effects
-			(font
-				(size 1.27 1.27)
-			)
+		(at 108.712 67.056 0)
+		(effects
+			(font
+				(size 1.27 1.27)
+			)
+			(justify left)
 		)
 	)
@@
 		)
 	)
-	(label "CLK3"
+	(label "CLK1"
 		(at 262.89 111.76 0)
 		(fields_autoplaced yes)
@@
 		)
 	)
-	(label "CLK4"
+	(label "CLK3"
 		(at 262.89 99.06 0)
 		(fields_autoplaced yes)
@@
 		)
 	)
-	(label "CLK1"
+	(label "CLK4"
 		(at 262.89 114.3 0)
 		(fields_autoplaced yes)

Commit message: messing with xtal
Parts:
- removed JP2: CD2, Jumper:SolderJumper-2_P1.3mm_Open_RoundedPad1.0x1.5mm, symbol Jumper:SolderJumper_2_Open
- removed JP3: CD1, Jumper:SolderJumper-2_P1.3mm_Open_RoundedPad1.0x1.5mm, symbol Jumper:SolderJumper_2_Open
Changed lines of the file:
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@@
 	)
 	(bus_entry
+		(at 275.59 106.68)
+		(size 2.54 2.54)
+		(stroke
+			(width 0)
+			(type default)
+		)
+	)
+	(bus_entry
 		(at 99.06 83.82)
 		(size 2.54 2.54)
@@
 	)
 	(bus_entry
+		(at 275.59 104.14)
+		(size 2.54 2.54)
+		(stroke
+			(width 0)
+			(type default)
+		)
+	)
+	(bus_entry
 		(at 110.49 115.57)
 		(size -2.54 -2.54)
@@
 	)
 	(bus_entry
-		(at 275.59 106.68)
-		(size 2.54 2.54)
-		(stroke
-			(width 0)
-			(type default)
-		)
-	)
-	(bus_entry
 		(at 66.04 116.84)
 		(size 2.54 2.54)
@@
 	)
 	(bus_entry
-		(at 275.59 104.14)
-		(size 2.54 2.54)
-		(stroke
-			(width 0)
-			(type default)
-		)
-	)
-	(bus_entry
 		(at 139.7 87.63)
 		(size -2.54 -2.54)
@@
 		)
 	)
+	(bus
+		(pts
+			(xy 278.13 106.68) (xy 278.13 109.22)
+		)
+		(stroke
+			(width 0)
+			(type default)
+		)
+	)
 	(wire
 		(pts
@@
 	(bus
 		(pts
-			(xy 278.13 109.22) (xy 278.13 111.76)
+			(xy 278.13 104.14) (xy 278.13 106.68)
 		)
 		(stroke
@@
 	(bus
 		(pts
-			(xy 278.13 106.68) (xy 278.13 109.22)
-		)
-		(stroke
-			(width 0)
-			(type default)
-		)
-	)
-	(bus
-		(pts
 			(xy 66.04 96.52) (xy 66.04 99.06)
 		)
@@
 	(wire
 		(pts
+			(xy 262.89 106.68) (xy 275.59 106.68)
+		)
+		(stroke
+			(width 0)
+			(type default)
+		)
+	)
+	(wire
+		(pts
 			(xy 95.25 134.62) (xy 99.06 134.62)
 		)
@@
 		)
 	)
+	(bus
+		(pts
+			(xy 278.13 109.22) (xy 278.13 111.76)
+		)
+		(stroke
+			(width 0)
+			(type default)
+		)
+	)
 	(wire
 		(pts
@@
 		)
 	)
-	(wire
-		(pts
-			(xy 270.51 104.14) (xy 275.59 104.14)
-		)
-		(stroke
-			(width 0)
-			(type default)
-		)
-	)
 	(bus
 		(pts
@@
 	(wire
 		(pts
+			(xy 262.89 104.14) (xy 275.59 104.14)
+		)
+		(stroke
+			(width 0)
+			(type default)
+		)
+	)
+	(wire
+		(pts
 			(xy 129.54 107.95) (xy 129.54 105.41)
 		)
@@
 		)
 	)
-	(wire
-		(pts
-			(xy 270.51 106.68) (xy 275.59 106.68)
-		)
-		(stroke
-			(width 0)
-			(type default)
-		)
-	)
 	(bus
 		(pts
@@
 	(bus
 		(pts
-			(xy 278.13 104.14) (xy 278.13 106.68)
-		)
-		(stroke
-			(width 0)
-			(type default)
-		)
-	)
-	(bus
-		(pts
 			(xy 195.58 110.49) (xy 195.58 107.95)
 		)
@@
 		)
 	)
-	(label "CD1"
-		(at 271.78 106.68 0)
-		(fields_autoplaced yes)
-		(effects
-			(font
-				(size 1.27 1.27)
-			)
-			(justify left bottom)
-		)
-	)
 	(label "WAIT"
 		(at 204.47 123.19 180)
@@
 		)
 	)
-	(label "CD2"
-		(at 271.78 104.14 0)
-		(fields_autoplaced yes)
-		(effects
-			(font
-				(size 1.27 1.27)
-			)
-			(justify left bottom)
-		)
-	)
 	(label "D13"
 		(at 95.25 63.5 0)
@@
 	)
 	(symbol
-		(lib_id "Jumper:SolderJumper_2_Open")
-		(at 266.7 106.68 0)
-		(unit 1)
-		(exclude_from_sim yes)
-		(in_bom no)
-		(on_board yes)
-		(dnp no)
-		(property "Reference" "JP3"
-			(at 266.7 100.33 0)
-			(effects
-				(font
-					(size 1.27 1.27)
-				)
-				(hide yes)
-			)
-		)
-		(property "Value" "CD1"
-			(at 264.16 105.41 0)
-			(effects
-				(font
-					(size 1.27 1.27)
-				)
-			)
-		)
-		(property "Footprint" "Jumper:SolderJumper-2_P1.3mm_Open_RoundedPad1.0x1.5mm"
-			(at 266.7 106.68 0)
-			(effects
-				(font
-					(size 1.27 1.27)
-				)
-				(hide yes)
-			)
-		)
-		(property "Datasheet" "~"
-			(at 266.7 106.68 0)
-			(effects
-				(font
-					(size 1.27 1.27)
-				)
-				(hide yes)
-			)
-		)
-		(property "Description" "Solder Jumper, 2-pole, open"
-			(at 266.7 106.68 0)
-			(effects
-				(font
-					(size 1.27 1.27)
-				)
-				(hide yes)
-			)
-		)
-		(pin "1"
-		)
-		(pin "2"
-		)
-		(instances
-			(project "devboard"
-				(path "/faa55760-cb03-4d07-a56c-933314735a7e"
-					(reference "JP3")
-					(unit 1)
-				)
-			)
-		)
-	)
-	(symbol
 		(lib_id "power:+5VD")
 		(at 81.915 156.21 0)
@@
 					(unit 1)
 				)
-			)
-		)
-	)
-	(symbol
-		(lib_id "Jumper:SolderJumper_2_Open")
-		(at 266.7 104.14 0)
-		(unit 1)
-		(exclude_from_sim yes)
-		(in_bom no)
-		(on_board yes)
-		(dnp no)
-		(property "Reference" "JP2"
-			(at 266.7 97.79 0)
-			(effects
-				(font
-					(size 1.27 1.27)
-				)
-				(hide yes)
-			)
-		)
-		(property "Value" "CD2"
-			(at 264.16 102.87 0)
-			(effects
-				(font
-					(size 1.27 1.27)
-				)
-			)
-		)
-		(property "Footprint" "Jumper:SolderJumper-2_P1.3mm_Open_RoundedPad1.0x1.5mm"
-			(at 266.7 104.14 0)
-			(effects
-				(font
-					(size 1.27 1.27)
-				)
-				(hide yes)
-			)
-		)
-		(property "Datasheet" "~"
-			(at 266.7 104.14 0)
-			(effects
-				(font
-					(size 1.27 1.27)
-				)
-				(hide yes)
-			)
-		)
-		(property "Description" "Solder Jumper, 2-pole, open"
-			(at 266.7 104.14 0)
-			(effects
-				(font
-					(size 1.27 1.27)
-				)
-				(hide yes)
-			)
-		)
-		(pin "1"
-		)
-		(pin "2"
-		)
-		(instances
-			(project ""
-				(path "/faa55760-cb03-4d07-a56c-933314735a7e"
-					(reference "JP2")
-					(unit 1)
-				)
